Commit message: edits for xacro and launch and urdf

File: urdf/edumip_my_robot.urdf (robot description, URDF)
Before this commit: robot edumip_my_robot, 3 links, 2 joints
Links:
- added link stripeL; visual box size=0.005 0.068 0.005
Joints:
- added joint stripe_jointL: type fixed, parent wheelL, child stripeL, origin xyz=0.0 0.0 0.0 rpy=0 0 0, axis 0 1 0
